File: sheet_output.kicad_sch (KiCad schematic)
At the start: 9 parts, among them J2 TRRS PJ-3X4S (CTIA, bottom-si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

Commit message: sch: add datasheet links, hide Datasheet/Description fields, remove sentinel text
- Filled 38 empty component Datasheet fields with LCSC product-page links (derived from the BOM part numbers); fixed D8's stale link (Kingbright KP-2012EC -> white KT-0805W / C34499). Existing manufacturer/distributor links kept.
- Hid the Datasheet and Description fields on all 53 placed components (most were previously shown, cluttering the canvas).
- Removed the 4 leftover sentinel text annotations.
- Netlist unchanged (check_sync: in sync, 53 comps / 46 nets).
Other:
- note removed: "claude-insert-below — sentinel for Edit anchors. DO NOT DELETE."
Changed lines of the file:
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@@
 		(comment 1 "Chunk 3: TRRS jack + output coupling + electret mic bias")
-	)
-	(text "claude-insert-below — sentinel for Edit anchors. DO NOT DELETE."
-		(exclude_from_sim no)
-		(at 191.77 22.098 0)
-		(effects
-			(font
-				(size 0.5 0.5)
-			)
-			(justify left top)
-		)
 	)
 	(wire
@@
 		)
 		(property "Value" "TRRS PJ-3X4S (CTIA, bottom-side)"
-			(at 243.332 110.236 0)
-			(show_name no)
-			(do_not_autoplace no)
-			(effects
-				(font
-					(size 1.27 1.27)
-				)
-				(justify right bottom)
+			(at 205.994 109.728 0)
+			(show_name no)
+			(do_not_autoplace no)
+			(effects
+				(font
+					(size 1.27 1.27)
+				)
+				(justify left bottom)
 			)
 		)
@@
 		(property "Datasheet" "https://www.sameskydevices.com/product/interconnect/connectors/audio-connectors/jacks/sj-3524-smt-tr"
 			(at 216.154 101.346 0)
+			(hide yes)
 			(show_name no)
 			(do_not_autoplace no)
@@
 		(property "Description" ""
 			(at 216.154 101.346 0)
+			(hide yes)
 			(show_name no)
 			(do_not_autoplace no)
@@
 		(dnp no)
 		(property "Reference" "R9"
-			(at 189.992 101.394 0)
+			(at 189.484 101.6 90)
 			(show_name no)
 			(do_not_autoplace no)
@@
 		)
 		(property "Value" "33R"
-			(at 189.992 107.394 0)
+			(at 189.992 107.442 90)
 			(show_name no)
 			(do_not_autoplace no)
@@
 			)
 		)
-		(property "Datasheet" ""
+		(property "Datasheet" "https://www.lcsc.com/product-detail/C25105.html"
 			(at 189.992 104.394 0)
+			(hide yes)
 			(show_name no)
 			(do_not_autoplace no)
@@
 		(property "Description" ""
 			(at 189.992 104.394 0)
+			(hide yes)
 			(show_name no)
 			(do_not_autoplace no)
@@
 		(dnp no)
 		(property "Reference" "R10"
-			(at 190.5 115.618 0)
+			(at 190.5 115.316 90)
 			(show_name no)
 			(do_not_autoplace no)
@@
 		)
 		(property "Value" "33R"
-			(at 190.5 121.618 0)
+			(at 190.5 121.666 90)
 			(show_name no)
 			(do_not_autoplace no)
@@
 			)
 		)
-		(property "Datasheet" ""
+		(property "Datasheet" "https://www.lcsc.com/product-detail/C25105.html"
 			(at 190.5 118.618 0)
+			(hide yes)
 			(show_name no)
 			(do_not_autoplace no)
@@
 		(property "Description" ""
 			(at 190.5 118.618 0)
+			(hide yes)
 			(show_name no)
 			(do_not_autoplace no)
@@
 		(dnp no)
 		(property "Reference" "C14"
-			(at 189.738 71.93 0)
+			(at 189.484 70.866 90)
 			(show_name no)
 			(do_not_autoplace no)
@@
 		)
 		(property "Value" "22uF"
-			(at 189.738 77.93 0)
+			(at 190.246 78.74 90)
 			(show_name no)
 			(do_not_autoplace no)
@@
 			)
 		)
-		(property "Datasheet" ""
+		(property "Datasheet" "https://www.lcsc.com/product-detail/C29277.html"
 			(at 189.738 74.93 0)
+			(hide yes)
 			(show_name no)
 			(do_not_autoplace no)
@@
 		(property "Description" ""
 			(at 189.738 74.93 0)
+			(hide yes)
 			(show_name no)
 			(do_not_autoplace no)
@@
 		(dnp no)
 		(property "Reference" "C15"
-			(at 189.738 58.214 0)
+			(at 189.992 57.404 90)
 			(show_name no)
 			(do_not_autoplace no)
@@
 		)
 		(property "Value" "22uF"
-			(at 189.738 64.214 0)
+			(at 190.5 64.77 90)
 			(show_name no)
 			(do_not_autoplace no)
@@
 			)
 		)
-		(property "Datasheet" ""
+		(property "Datasheet" "https://www.lcsc.com/product-detail/C29277.html"
 			(at 189.738 61.214 0)
+			(hide yes)
 			(show_name no)
 			(do_not_autoplace no)
@@
 		(property "Description" ""
 			(at 189.738 61.214 0)
+			(hide yes)
 			(show_name no)
 			(do_not_autoplace no)
@@
 		(dnp no)
 		(property "Reference" "C12"
-			(at 240.35 58.482 0)
+			(at 240.538 57.404 90)
 			(show_name no)
 			(do_not_autoplace no)
@@
 		)
 		(property "Value" "1uF"
-			(at 240.35 64.482 0)
+			(at 240.538 65.532 90)
 			(show_name no)
 			(do_not_autoplace no)
@@
 			)
 		)
-		(property "Datasheet" ""
+		(property "Datasheet" "https://www.lcsc.com/product-detail/C52923.html"
 			(at 240.35 61.482 0)
+			(hide yes)
 			(show_name no)
 			(do_not_autoplace no)
@@
 		(property "Description" ""
 			(at 240.35 61.482 0)
+			(hide yes)
 			(show_name no)
 			(do_not_autoplace no)
@@
 		(dnp no)
 		(property "Reference" "C20"
-			(at 189.738 85.646 0)
+			(at 189.738 85.09 90)
 			(show_name no)
 			(do_not_autoplace no)
@@
 		)
 		(property "Value" "1uF"
-			(at 189.738 91.646 0)
+			(at 190.246 92.71 90)
 			(show_name no)
 			(do_not_autoplace no)
@@
 			)
 		)
-		(property "Datasheet" ""
+		(property "Datasheet" "https://www.lcsc.com/product-detail/C52923.html"
 			(at 189.738 88.646 0)
+			(hide yes)
 			(show_name no)
 			(do_not_autoplace no)
@@
 		(property "Description" ""
 			(at 189.738 88.646 0)
+			(hide yes)
 			(show_name no)
 			(do_not_autoplace no)
@@
 		(dnp no)
 		(property "Reference" "R7"
-			(at 223.774 70.406 0)
+			(at 223.774 70.358 90)
 			(show_name no)
 			(do_not_autoplace no)
@@
 		)
 		(property "Value" "2.2k (mic bias)"
-			(at 223.774 76.406 0)
+			(at 225.298 76.962 90)
 			(show_name no)
 			(do_not_autoplace no)
@@
 			)
 		)
-		(property "Datasheet" ""
+		(property "Datasheet" "https://www.lcsc.com/product-detail/C25879.html"
 			(at 223.774 73.406 0)
+			(hide yes)
 			(show_name no)
 			(do_not_autoplace no)
@@
 		(property "Description" ""
 			(at 223.774 73.406 0)
+			(hide yes)
 			(show_name no)
 			(do_not_autoplace no)
@@
 		(dnp no)
 		(property "Reference" "C13"
-			(at 257.27 75.66 0)
-			(show_name no)
-			(do_not_autoplace no)
-			(effects
-				(font
-					(size 1.27 1.27)
-				)
-				(justify left)
+			(at 257.048 69.596 90)
+			(show_name no)
+			(do_not_autoplace no)
+			(effects
+				(font
+					(size 1.27 1.27)
+				)
+				(justify right)
 			)
 		)
 		(property "Value" "1uF (bias filter)"
-			(at 254.27 75.66 0)
-			(show_name no)
-			(do_not_autoplace no)
-			(effects
-				(font
-					(size 1.27 1.27)
-				)
-				(justify left)
+			(at 262.382 77.978 90)
+			(show_name no)
+			(do_not_autoplace no)
+			(effects
+				(font
+					(size 1.27 1.27)
+				)
+				(justify right)
 			)
 		)
@@
 			)
 		)
-		(property "Datasheet" ""
+		(property "Datasheet" "https://www.lcsc.com/product-detail/C52923.html"
 			(at 255.27 73.66 0)
+			(hide yes)
 			(show_name no)
 			(do_not_autoplace no)
@@
 		(property "Description" ""
 			(at 255.27 73.66 0)
-			(show_name no)
-			(do_not_autoplace no)
+			(hide yes)
+			(show_name no)
+			(do_not_autoplace no)
